File: bldc motor controller.kicad_sch (KiCad schematic)
At the start: 47 parts

Commit message: Almost done design, need to add mounting holes I think
Parts:
- C19: footprint Capacitor_SMD:C_0402_1005Metric -> Capacitor_SMD:C_01005_0402Metric
- U2: footprint bldc-motor-footprints:CONN-SMD_4P-P1.25_SM04B-GHS-TB-LF-SN -> Connector_JST:JST_ACH_BM04B-ACHSS-A-GAN-ETF_1x04-1MP_P1.20mm_Vertical
- U7: footprint bldc-motor-footprints:CONN-SMD_SM02B-GHS-TB-LF-SN -> Connector_JST:JST_GH_BM02B-GHS-TBT_1x02-1MP_P1.25mm_Vertical
- U8: footprint Button_Switch_THT:SW_Slide-03_Wuerth-WS-SLTV_10x2.5x6.4_P2.54mm -> Connector_PinHeader_2.54mm:PinHeader_1x03_P2.54mm_Vertical
Connections:
- net PHASE-A: now also U8.1; no longer U8.2
- net PHASE-B: now also U8.2; no longer U8.1
- net TI_AVDD: now also C10.2, U1.1 (CP)
Changed lines of the file:
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@@
 	(wire
 		(pts
-			(xy 261.62 100.33) (xy 261.62 101.6)
-		)
-		(stroke
-			(width 0)
-			(type default)
-		)
-	)
-	(wire
-		(pts
 			(xy 74.93 143.51) (xy 74.93 135.89)
 		)
@@
 	(wire
 		(pts
+			(xy 261.62 97.79) (xy 261.62 101.6)
+		)
+		(stroke
+			(width 0)
+			(type default)
+		)
+	)
+	(wire
+		(pts
 			(xy 25.4 82.55) (xy 25.4 76.2)
 		)
@@
 	(global_label "PHASE-B"
 		(shape input)
-		(at 261.62 137.16 90)
+		(at 259.08 137.16 90)
 		(fields_autoplaced yes)
 		(effects
@@
 		)
 		(property "Intersheetrefs" "${INTERSHEET_REFS}"
-			(at 261.62 125.2848 90)
+			(at 259.08 125.2848 90)
 			(effects
 				(font
@@
 	(global_label "PHASE-A"
 		(shape input)
-		(at 259.08 137.16 90)
+		(at 261.62 137.16 90)
 		(fields_autoplaced yes)
 		(effects
@@
 		)
 		(property "Intersheetrefs" "${INTERSHEET_REFS}"
-			(at 259.08 125.4662 90)
+			(at 261.62 125.4662 90)
 			(effects
 				(font
@@
 			)
 		)
-		(property "Footprint" "Capacitor_SMD:C_0402_1005Metric"
+		(property "Footprint" "Capacitor_SMD:C_01005_0402Metric"
 			(at 74.93 146.05 0)
 			(effects
@@
 			)
 		)
-		(property "Footprint" "bldc-motor-footprints:CONN-SMD_SM02B-GHS-TB-LF-SN"
+		(property "Footprint" "Connector_JST:JST_GH_BM02B-GHS-TBT_1x02-1MP_P1.25mm_Vertical"
 			(at 126.746 136.906 0)
 			(effects
@@
 			)
 		)
-		(property "Footprint" "bldc-motor-footprints:CONN-SMD_4P-P1.25_SM04B-GHS-TB-LF-SN"
+		(property "Footprint" "Connector_JST:JST_ACH_BM04B-ACHSS-A-GAN-ETF_1x04-1MP_P1.20mm_Vertical"
 			(at 204.724 172.466 0)
 			(effects
@@
 			)
 		)
-		(property "Footprint" "Button_Switch_THT:SW_Slide-03_Wuerth-WS-SLTV_10x2.5x6.4_P2.54mm"
+		(property "Footprint" "Connector_PinHeader_2.54mm:PinHeader_1x03_P2.54mm_Vertical"
 			(at 229.87 142.24 0)
 			(effects

Commit message: Power Ground Signal Ground Seperate
Parts:
- C21, C23: value C_Small -> 100nF
- C22: value C_Small -> 10uF
Connections:
- net +3.3VA: no longer C1.2, C8.2, C9.2, CN1.1, R6.2, U1.2 (VM), U2.4, U2.5, U2.6, U4.2 (GND), U7.3, U7.4
- new net -BATT: C1.2, C8.2, C9.2, CN1.1, R6.2, U1.2 (VM), U4.2 (GND)
- new net GND1: U2.4

Commit message: 4 layer nice looking board
Parts:
- removed U2: ~, Connector_JST:JST_ACH_BM04B-ACHSS-A-GAN-ETF_1x04-1MP_P1.20mm_Vertical, symbol bldc controller:SM04B-GHS-TB(LF)(SN)
- added J1: Conn_01x04_Pin, Connector_PinHeader_1.00mm:PinHeader_1x04_P1.00mm_Vertical, symbol Connector:Conn_01x04_Pin
- added NT1: NetTie_2, NetTie:NetTie-2_SMD_Pad0.5mm, symbol Device:NetTie_2
- C22: footprint Capacitor_SMD:C_01005_0402Metric -> Capacitor_SMD:C_0603_1608Metric
- L1: Supplier Part (none) -> C7461351
- LED1: footprint bldc-motor-footprints:LED0603-RD -> LED_SMD:LED_0603_1608Metric
- U1: value ~ -> C47023655
- U3: value ~ -> C529358
- U6: value ~ -> C126671; Supplier LCSC -> JLC
- U8: now not fitted
- renumbered CN1 to -BAT+1
Connections:
- net +3.3V: now also J1.3 (Pin_3)
- net +3.3VA: now also J1.4 (Pin_4), NT1.2
- net -BATT: now also NT1.1
- net UART_RX: now also J1.2 (Pin_2)
- net UART_TX: now also J1.1 (Pin_1)
- no-connect marks 0 -> 12

Commit message: resistor for current sense did not exist
Parts:
- R2, R3, R4: footprint Resistor_SMD:R_01005_0402Metric -> Resistor_SMD:R_0201_0603Metric
Changed lines of the file:
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@@
 			)
 		)
-		(property "Footprint" "Resistor_SMD:R_01005_0402Metric"
+		(property "Footprint" "Resistor_SMD:R_0201_0603Metric"
 			(at 172.466 53.086 90)
 			(effects
@@
 			)
 		)
-		(property "Footprint" "Resistor_SMD:R_01005_0402Metric"
+		(property "Footprint" "Resistor_SMD:R_0201_0603Metric"
 			(at 175.006 65.786 90)
 			(effects
@@
 			)
 		)
-		(property "Footprint" "Resistor_SMD:R_01005_0402Metric"
+		(property "Footprint" "Resistor_SMD:R_0201_0603Metric"
 			(at 175.006 77.216 90)
 			(effects
