File: bldc motor controller.kicad_pcb (KiCad board)
At the start: 4 copper layers, 26 x 26 mm, 61 parts, among them J1 Conn_01x04_Pin, J2 Conn_01x02, M2 MountingHole_2.2mm_M2_DIN965_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, U1 C47023655, U10 STM32G431KBUx, U2 LSM6DSV16XTR, U6 LIS2MDLTR

Commit message: final review time
Parts:
- R12, R5: value 10kOhm -> 10k
- U1: value C47023655 -> ~
Connections:
- U9 pad 9: unconnected-(U9-PAD-Pad9) -> GND
Routing:
- net GND: track 102.2 -> 127.6 mm, vias 7 -> 12
- net -BATT: track 52.4 -> 54.2 mm
- net +3.3V: track 186.8 -> 187.6 mm, vias 8 -> 9
- net SOA: track 7.42 -> 6.66 mm
- added copper zone on B.Cu, net GND
- added copper zone on F.Cu, net GND
