File: _autosave-bldc motor controller.kicad_pcb (KiCad board)
At the start: 4 copper layers, 26 x 26 mm, 61 parts, among them J1 Conn_01x04_Pin, J2 Conn_01x02, M2 MountingHole_2.2mm_M2_DIN965_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, U10 STM32G431KBUx, U2 LSM6DSV16XTR, U6 LIS2MDLTR

Commit message: and I think I am done! oh boy oh boy
Parts:
- removed C28, C29: 10 uf X5R 50v, Capacitor_SMD:C_0603_1608Metric
- C1: value 2.2UF -> 2.2UF X7R 50V; footprint Capacitor_SMD:C_1206_3216Metric -> Capacitor_SMD:C_0805_2012Metric
- C9: footprint Capacitor_SMD:C_0603_1608Metric -> Capacitor_SMD:C_1206_3216Metric; moved to B.Cu
- moved C9 11.9 mm to (142.2, 94.6), turned to 180 degrees
- moved C8 6.25 mm to (139.4, 92.6)
- moved C1 5.55 mm to (138.0, 98.1), turned to 0 degrees
- moved R6 0.08 mm to (137.9, 96.4)
Connections:
- U6 pad 11: unconnected-(U6-NC2-Pad11) -> GND
- U6 pad 12: unconnected-(U6-NC3-Pad12) -> GND
- U6 pad 2: unconnected-(U6-NC1-Pad2) -> GND
Routing:
- net GND: track 155.4 -> 159.0 mm
- net -BATT: track 51.9 -> 49.4 mm
- net +BATT: track 54.0 -> 52.7 mm
- net +3.3V: track 191.9 -> 190.7 mm
- net Net-(U4-SW): track 9.02 -> 7.90 mm
- added copper zone on F.Cu, net +3.3V
